Commit message: Imported upstream version '0.1.1' of 'upstream'

File: flir_ptu_description/urdf/d46.urdf.xacro (robot description, xacro)
@@ -54,7 +54,7 @@
     <joint name="${name}_pan" type="revolute">
       <parent link="${name}_pan_link" />
-      <origin xyz="0 0 0.066" rpy="-1.5708 0 0" />
+      <origin xyz="0 0 0.066" rpy="1.5708 0 0" />
       <child link="${name}_tilt_link" />
-      <axis xyz="0 1 0" />
+      <axis xyz="0 -1 0" rpy="3.14159 0 0" />
       <limit lower="${-pan_range}" upper="${pan_range}"
              effort="${joint_effort}" velocity="${pan_velocity}" />

Commit message: Imported upstream version '0.1.4' of 'upstream'

File: flir_ptu_description/urdf/d46.urdf.xacro (robot description, xacro)
@@ -54,8 +54,8 @@
     <joint name="${name}_pan" type="revolute">
       <parent link="${name}_pan_link" />
-      <origin xyz="0 0 0.066" rpy="1.5708 0 0" />
+      <origin xyz="0 0 0.066" rpy="-1.5708 0 0" />
       <child link="${name}_tilt_link" />
-      <axis xyz="0 -1 0" rpy="3.14159 0 0" />
-      <limit lower="${-pan_range}" upper="${pan_range}"
+      <axis xyz="0 1 0" rpy="0 0 0" />
+      <limit lower="${pan_range}" upper="${-pan_range}"
              effort="${joint_effort}" velocity="${pan_velocity}" />
     </joint>

File: flir_ptu_description/urdf/example.urdf.xacro (robot description, xacro)
@@ -2,7 +2,9 @@
 <robot name="ptu_d46"
        xmlns:xacro="http://ros.org/wiki/xacro">
+  <link name="base_link" />
+  <!-- Include and invoke the macro which creates a D46 -->
   <xacro:include filename="d46.urdf.xacro" />
   <ptu_d46 name="ptu" />
-  <link name="base_link" />
+  <!-- Create a fixed joint to connect the PTU to the rest of the robot -->
   <joint name="base_to_ptu_base" type="fixed">
     <parent link="base_link"/>
@@ -10,3 +12,5 @@
     <origin xyz="0 0 0"/>
   </joint>
+  <!-- If you had a lidar or some other device mounted on the PTU, you would create another
+       fixed joint here between the ptu_mount link and the origin of the device. -->
 </robot>
